File: telecommande/telecommande.kicad_pcb (KiCad board)
At the start: 2 copper layers, 45 x 53 mm, 43 parts, among them J1 Conn_01x08_Male, J2 Conn_01x02_Male, J3 Conn_01x04_Male, J4 Conn_01x04_Male, J5 Conn_01x06_Male, J6 Screw_Terminal_01x02, J7 Screw_Terminal_01x02, J8 Conn_01x01_Male, K1 ATX203, Q1 BS170, SW1 SW_MEC_5E, U1 L78L05_TO92, U2 PIC18F26K80_ISS, U3 24LC1026-I_P, U4 L7812, Y1 Crystal 16MHz

Commit message: add came
Parts:
- added J10: Conn_01x04_Female, Connector_PinSocket_2.54mm:PinSocket_1x04_P2.54mm_Vertical, F.Cu at (89.9, 119.4)
- added J9: Conn_01x03_Female, Connector_PinSocket_2.54mm:PinSocket_1x03_P2.54mm_Vertical, F.Cu at (92.5, 84.1)
- D3: footprint Diode_THT:D_DO-41_SOD81_P10.16mm_Horizontal -> Diode_THT:D_DO-41_SOD81_P7.62mm_Horizontal
- J2: footprint Connector_PinSocket_2.54mm:PinSocket_1x02_P2.54mm_Vertical -> Connector_PinHeader_2.54mm:PinHeader_1x02_P2.54mm_Vertical
- J3: value Conn_01x04_Male -> Conn_01x04_Female
- J4: value Conn_01x04_Male -> Conn_01x02_Female; footprint Connector_PinSocket_2.54mm:PinSocket_1x04_P2.54mm_Vertical -> Connector_PinSocket_2.54mm:PinSocket_1x02_P2.54mm_Vertical
- moved D3 37.6 mm to (95.8, 75.4), turned to 180 degrees
- moved J4 12.0 mm to (92.5, 107.7)
- moved Q1 0.76 mm to (99.3, 89.2)
Connections:
- J4 pad 1: GND -> /ANT
- J4 pad 2: /RX -> GND
Routing:
- net Net-(C8-Pad1): track 11.5 -> 48.2 mm
- net Net-(D3-Pad2): track 35.8 -> 6.92 mm
- net /RX: track 48.5 -> 72.8 mm, vias 0 -> 1
- net /ANT: track 39.5 -> 51.3 mm
- net /VDD: track 115.0 -> 120.9 mm
- net GND: track 96.3 -> 100.9 mm, vias 2 -> 3
- net /TVDD: track 14.4 -> 11.0 mm
- net /12VR: track 72.3 -> 74.8 mm
- net Net-(C7-Pad2): track 19.9 -> 18.8 mm
- net /LED: track 37.9 -> 36.8 mm
- net /Rel1: track 18.3 -> 18.9 mm
Other:
- board text added: "Réc RFM210LCF-A"
- board text added: "Récept. télécommandes"
- board text removed: "Décodeur NiceflorS"

Commit message: V2
Parts:
- added J11: Conn_01x04_Female, Connector_PinSocket_2.54mm:PinSocket_1x04_P2.54mm_Vertical, F.Cu at (89.9, 90.7)
- R4, R5, R7: value 220 -> 90
- R6: value 220 -> 90; moved to B.Cu
- moved R6 2.54 mm to (119.4, 108.0)
- moved R7 2.29 mm to (119.4, 110.2)
- moved U4 1.52 mm to (99.6, 121.2)
- moved C4 1.02 mm to (110.0, 118.6)
- moved U1 1.02 mm to (108.7, 120.7)
- moved D5 0.51 mm to (116.3, 116.3)
Connections:
- J5 pad 3: /RX1 -> /TX1
- J5 pad 4: /TX1 -> /RX1
- U2 pad 5: (no net) -> /Enable
Routing:
- net /RX: track 72.8 -> 97.8 mm
- net /Enable: track 0.00 -> 19.6 mm
- net /VDD: track 120.9 -> 128.9 mm
- net GND: track 100.9 -> 94.2 mm
- net Net-(R7-Pad2): track 7.57 -> 10.8 mm
- net Net-(D3-Pad2): track 6.92 -> 4.82 mm
- net /VCC: track 22.5 -> 24.1 mm
- net /ANT: track 51.3 -> 52.8 mm
- net Net-(C8-Pad1): track 48.2 -> 49.4 mm
- net /RX1: track 2.30 -> 2.93 mm
- net Net-(R6-Pad2): track 7.82 -> 7.23 mm, vias 0 -> 1
- net /TX1: track 2.30 -> 2.81 mm
Other:
- board text added: "CTS"
- board text added: "HM-R433"
- board text added: "RFM210LCF-A"
- board text added: "RXB6"
- board text removed: "RTS"
- board text removed: "Réc RFM210LCF-A"
- board text removed: "Récepteur RXB6"
